File: zynq.kicad_sch (KiCad schematic)
At the start: 1 part, among them IC1 XC7Z020-2CLG484I

Commit message: power + GND work, updates
Parts:
- removed IC1: XC7Z020-2CLG484I, BGA484C80P22X22_1900X1900X160, symbol zynq:XC7Z020-2CLG484I
Other:
- added sheet PL (PL.kicad_sch)
- added sheet PS (PS.kicad_sch)
- added sheet Power (power.kicad_sch)
- added sheet Power1 (power1.kicad_sch)
